File: hardware/JULIAN FINAL.kicad_pcb (KiCad board)
At the start: 2 copper layers, 99 x 69 mm, 13 parts, among them J2 Jack-DC, J4 HEADER_4, M1 Motor_Servo_Futaba_J

Commit message: Add files via upload
Parts:
- moved C1 1.70 mm to (149.7, 105.5)
- moved J2 0.60 mm to (78.0, 77.0)
Connections:
- net Net-(D1-A) renamed 12V
- ? pad 1: Net-(J3-Pin_2) -> 5V
- C1 pad 2: Net-(G´pio12-5V) -> 5V
- C3 pad 2: Net-(G´pio12-5V) -> 5V
- G´pio12 pad 10: (no net) -> GND
- G´pio12 pad 12: (no net) -> Net-(G´pio12-GPIO13)
- G´pio12 pad 2: (no net) -> Net-(G´pio12-GPIO3)
- G´pio12 pad 3: (no net) -> Net-(G´pio12-GPIO3)
- G´pio12 pad 9: (no net) -> 5V
- J2 pad 2: Net-(J1-Pin_2) (its old number) -> PGND
- J4 pad 1: Net-(G´pio12-5V) -> 5V
- J4 pad 2: Net-(G´pio12-GPIO1) (its old number) -> Net-(G´pio12-GPIO3)
- M1 pad 1: Net-(G´pio12-GPIO12) -> Net-(G´pio12-GPIO13)
- ds pad 1: Net-(J1-Pin_2) (its old number) -> PGND
Routing:
- net 5V: track 0.00 -> 155.2 mm
- net Net-(J3-Pin_2): track 122.1 -> 0.00 mm
- net PGND: track 0.00 -> 47.9 mm
- net Net-(J1-Pin_2) (its old number): track 47.9 -> 0.00 mm
- net Net-(G´pio12-GPIO1): track 45.2 -> 0.00 mm
- net Net-(G´pio12-GPIO1) (its old number): track 38.7 -> 0.00 mm
- net Net-(G´pio12-GPIO3): track 0.00 -> 35.4 mm
- net Net-(G´pio12-GPIO13): track 0.00 -> 32.8 mm
- net Net-(G´pio12-GPIO12): track 30.4 -> 0.00 mm
- net Net-(G´pio12-5V): track 21.5 -> 0.00 mm
- net Net-(C1-Pad1): track 62.5 -> 63.2 mm
