File: hardware/JULIAN FINAL.kicad_sch (KiCad schematic)
At the start: 11 parts, among them J1 Screw_Terminal_01x02, J2 Jack-DC, J3 Screw_Terminal_01x02, J4 HEADER_4, M1 Motor_Servo_Futaba_J

Commit message: Add files via upload
Parts:
- J1: footprint EESTN5:BORNERA2_AZUL -> Connector_PinHeader_1.27mm:PinHeader_1x02_P1.27mm_Vertical
Connections:
- net at M1.1 (PWM): now also G´pio12.P$12 (GPIO13); no longer G´pio12.P$11 (GPIO12)
Other:
- moved on the sheet: J2
Changed lines of the file:
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@@
 	(wire
 		(pts
-			(xy 115.062 87.63) (xy 125.73 87.63)
+			(xy 114.3 87.63) (xy 125.73 87.63)
 		)
 		(stroke
@@
 	(wire
 		(pts
+			(xy 220.726 87.63) (xy 220.726 91.44)
+		)
+		(stroke
+			(width 0)
+			(type default)
+		)
+	)
+	(wire
+		(pts
 			(xy 157.226 101.092) (xy 200.66 101.092)
 		)
@@
 	(wire
 		(pts
+			(xy 109.22 58.42) (xy 109.982 58.42)
+		)
+		(stroke
+			(width 0)
+			(type default)
+		)
+	)
+	(wire
+		(pts
 			(xy 148.59 83.566) (xy 148.59 85.09)
 		)
@@
 	(wire
 		(pts
-			(xy 115.062 87.63) (xy 115.062 57.912)
+			(xy 114.3 87.63) (xy 114.3 54.61)
 		)
 		(stroke
@@
 	(wire
 		(pts
+			(xy 196.85 87.63) (xy 220.726 87.63)
+		)
+		(stroke
+			(width 0)
+			(type default)
+		)
+	)
+	(wire
+		(pts
 			(xy 199.39 70.612) (xy 159.512 70.612)
 		)
@@
 	(wire
 		(pts
-			(xy 109.982 57.912) (xy 109.982 58.928)
+			(xy 109.22 54.61) (xy 109.22 58.42)
 		)
 		(stroke
@@
 	(wire
 		(pts
-			(xy 196.85 90.17) (xy 219.456 90.17)
-		)
-		(stroke
-			(width 0)
-			(type default)
-		)
-	)
-	(wire
-		(pts
 			(xy 159.512 70.612) (xy 159.512 82.55)
 		)
@@
 	(wire
 		(pts
+			(xy 220.726 91.44) (xy 219.456 91.44)
+		)
+		(stroke
+			(width 0)
+			(type default)
+		)
+	)
+	(wire
+		(pts
+			(xy 219.456 91.44) (xy 219.456 90.17)
+		)
+		(stroke
+			(width 0)
+			(type default)
+		)
+	)
+	(wire
+		(pts
 			(xy 219.456 101.346) (xy 237.236 101.346)
 		)
@@
 		(pts
 			(xy 148.59 100.33) (xy 153.67 100.33)
+		)
+		(stroke
+			(width 0)
+			(type default)
+		)
+	)
+	(wire
+		(pts
+			(xy 109.982 58.42) (xy 109.982 58.928)
 		)
 		(stroke
@@
 	(symbol
 		(lib_id "Connector:Jack-DC")
-		(at 112.522 50.292 270)
+		(at 111.76 46.99 270)
 		(unit 1)
 		(exclude_from_sim no)
@@
 		(fields_autoplaced yes)
 		(property "Reference" "J2"
-			(at 117.348 49.0219 90)
+			(at 116.586 45.7199 90)
 			(effects
 				(font
@@
 		)
 		(property "Value" "Jack-DC"
-			(at 117.348 51.5619 90)
+			(at 116.586 48.2599 90)
 			(effects
 				(font
@@
 		)
 		(property "Footprint" "Connector_BarrelJack:BarrelJack_Horizontal"
-			(at 111.506 51.562 0)
+			(at 110.744 48.26 0)
 			(effects
 				(font
@@
 		)
 		(property "Datasheet" "~"
-			(at 111.506 51.562 0)
+			(at 110.744 48.26 0)
 			(effects
 				(font
@@
 		)
 		(property "Description" "DC Barrel Jack"
-			(at 112.522 50.292 0)
+			(at 111.76 46.99 0)
 			(effects
 				(font
@@
 			)
 		)
-		(property "Footprint" "EESTN5:BORNERA2_AZUL"
+		(property "Footprint" "Connector_PinHeader_1.27mm:PinHeader_1x02_P1.27mm_Vertical"
 			(at 130.81 85.09 0)
 			(effects
